File: pocket-reform-motherboard/pocket-reform-motherboard.kicad_sch (KiCad schematic)
At the start: 372 parts, among them J1 CHARGER, J10 1-2199230-6, J11 Conn_01x33, J12 2199230-5, J13 FH35C-31S-0.3HW(50), J14 USB_C_Receptacle, J15 CONN_SPK, J16 SAMTEC_TSM-106-02-X-SH-A, J17 POWSW, J18 CONN_HEAD, J2 DM3AT-SF-PEJM5, J20 QWIIC, J3 USB_C_Receptacle, J4 09452812561, J5 SYSCTL, J6 USB_INT1, J61 UART, J7 HDMI_D_1.4, J8 SIM_Card, J9 Conn_01x20, SW1 SW_DIP_x01, SW2 RESET, U1 reform2-som-connector, U10 W25Q32JVSS, U11 PCF8523T, U12 AP22615AWU-7, U13 TXS0108EPW, U14 SN74AVC1T45, U15 TPD4E02B04DQA, U16 TPD4E02B04DQA, U17 TPD12S521, U18 TLV320AIC3100, U19 TPD4E02B04DQA, U2 TS3USB30EDGSR, U20 TPD4E02B04DQA, U21 TPD4E02B04DQA, U22 TPD4E02B04DQA, U23 FUSB302BMPX, U24 TXS0108EPW, U25 TUSB8041, U26 74HC573, U27 TVS2200DRV, U28 LM62460, U29 TPS62177DQC, U3 LM2830XQMFE/NOPB, U30 TS3USB30EDGSR, U31 TS3USB30EDGSR, U32 AP22615AWU-7, U33 AT24CS02-STUM, U34 PCA9536DP, U35 TMUXHS4446RETR, U4 TLV1117-18, U5 LM73100RPWR, U6 LM62460, U7 74LVC1G34, U8 RP2040, U9 TPS7A0533PDBZ, Y1 24MHz, Y2 12MHz 12pF, Y3 32.768 kHz

Commit message: mb1.5: routing WIP
Parts:
- removed C109: 0.1uF, Capacitor_SMD:C_0402_1005Metric, symbol Device:C_Small
- removed FB6: 100@100MHz 3A, Inductor_SMD:L_0603_1608Metric, symbol pocket-reform-motherboard-rescue:Ferrite_Bead_Small-Device
- removed R50: 0, Resistor_SMD:R_0402_1005Metric, symbol Device:R_Small
- removed U26: 74HC573, Package_SO:TSSOP-20_4.4x6.5mm_P0.65mm, symbol 74xx:74LS573
- added C141, C142, C143, C144, C145, C148: 0.1uF, Capacitor_SMD:C_0402_1005Metric, symbol Device:C_Small
- added C146: 4.7uF, Capacitor_SMD:C_0402_1005Metric, symbol Device:C_Small
- added C147: 1uF, Capacitor_SMD:C_0402_1005Metric, symbol Device:C_Small
- added R128, R130, R131, R134, R135, R138: 10k, Resistor_SMD:R_0402_1005Metric, symbol Device:R_Small
- added R129: 6.8k, Resistor_SMD:R_0402_1005Metric, symbol Device:R_Small
- added R132, R137: 2.2k, Resistor_SMD:R_0402_1005Metric, symbol Device:R_Small
- added R133, R136, R139: 0, Resistor_SMD:R_0402_1005Metric, symbol Device:R_Small
- added SW3: RESET, Button_Switch_SMD:SW_Push_1P1T_NO_CK_KMR2, symbol Switch:SW_SPST
- added TP7: UUART_SUSPEND, TestPoint:TestPoint_Pad_D1.0mm, symbol Connector:TestPoint
- added TP8: UUART_WAKEUP, TestPoint:TestPoint_Pad_D1.0mm, symbol Connector:TestPoint
- added TP9: UUART_nPOWER, TestPoint:TestPoint_Pad_D1.0mm, symbol Connector:TestPoint
- added U36: AP22615AWU-7, Package_TO_SOT_SMD:SOT-23-6, symbol Regulator_Linear:AP22615AWU
- added U37: TS3USB30EDGSR, Package_SO:VSSOP-10_3x3mm_P0.5mm, symbol Interface_USB:TS3USB30EDGSR
- added U38: CY7C65215-32LTXI, Package_DFN_QFN:QFN-32-1EP_5x5mm_P0.5mm_EP3.45x3.45mm, symbol Interface_USB:CY7C65215-32LTXI
- added U39: PCA9557RGVR, Package_DFN_QFN:Texas_RSA_VQFN-16-1EP_4x4mm_P0.65mm_EP2.7x2.7mm, symbol Interface_Expansion:PCA9557BS
- R21, R74, R78, R88: now not fitted
- R44: value 0 -> 10k; LCSC C242160 -> C60490; Manufacturer Panasonic -> Yageo; Manufacturer_No ERJ2GE0R00X -> RC0402FR-0710KL
- R45: value 0 -> 1k
- U35: footprint TMUXHS4446RETR:IC_TMUXHS4446RETR -> footprints:IC_TMUXHS4446RETR
Connections:
- net 5V_ENABLE is gone; now on an unnamed net: U8.37 (GPIO25)
- net +3V3: now also C141.1, R128.2, R136.2, U36.6 (IN)
- net 1V1_ENABLE_L: now also U39.8 (IO3)
- net 3V3_ENABLE_L: now also U39.7 (IO2)
- net 5V_ENABLE_L: now also U39.5 (IO1)
- net GND: now also C141.2, C142.2, C143.2, C144.2, C145.2, C146.2, C147.2, C148.2, R129.2, R130.1, SW3.2 (B), U36.2 (GND), U37.5 (GND), U38.17 (VSSD), U38.20 (VSSD), U38.24 (VSSA), U38.4 (VSSD), U39.2 (A1), U39.3 (A2), U39.6 (VSS); no longer R46.2
- net IMX_UART1_RX: now also R134.2, U38.30 (SCB0_4/GPIO_5)
- net IMX_UART1_TX: now also U38.2 (SCB0_0/GPIO_8)
- net IMX_UART2_RX: now also R135.2, U38.6 (SCB1_1/GPIO_11)
- net IMX_UART2_TX: now also U38.5 (SCB1_0/GPIO_10)
- net IMX_WAKE: now also U8.30 (GPIO19); no longer R45.2
- net LPC_MISO: now also U8.14 (GPIO11)
- net LPC_MOSI: now also U8.11 (GPIO8); no longer R44.2
- net RP_SCL0: now also U39.15 (SCL)
- net RP_SDA0: now also U39.16 (SDA)
- net USBH_2A_RXN: now also U35.16 (SSRX+); no longer U35.17 (SSRX-)
- net USBH_2A_RXP: now also U35.17 (SSRX-); no longer U35.16 (SSRX+)
- net USBH_2B_RXN: no longer U25.29 (USB_SSRXP_DN4)
- net USBH_2B_RXP: no longer U25.30 (USB_SSRXM_DN4)
- net USBH_2B_TXN: no longer U25.26 (USB_SSTXP_DN4)
- net USBH_2B_TXP: no longer U25.27 (USB_SSTXM_DN4)
- net USBH_2_DN: now also U37.8 (D1-); no longer J14.A7 (D-), J14.B7 (D-), U15.4 (IO3), U15.7 (IO3)
- net USBH_2_DP: now also U37.2 (D1+); no longer J14.A6 (D+), J14.B6 (D+), U15.5 (IO4), U15.6 (IO4)
- net USBM1_AC_RXN: now also U35.25 (CRX1+); no longer U35.24 (CRX1-)
- net USBM1_AC_RXP: now also U35.24 (CRX1-); no longer U35.25 (CRX1+)
- net USBM1_AC_TXN: now also C90.2; no longer C92.2
- net USBM1_AC_TXP: now also C92.2; no longer C90.2
- net USBM2_AC_RXN: now also U35.34 (CRX2+); no longer U35.33 (CRX2-)
- net USBM2_AC_RXP: now also U35.33 (CRX2-); no longer U35.34 (CRX2+)
- net USWITCH_OFF: now also U37.9 (~{OE}), U39.12 (IO7); no longer R118.2
- net VCC: now also R44.1, C142.1, C143.1, C144.1, C148.1, R131.2, R132.1, R133.1, R137.1, U39.14 (VDD)
- net ~{DISP_RESET_L}: now also U39.9 (IO4)
- net USBM1_TXN: now reaches C92.1, U35.27 (CTX1-)
- net USBM1_TXP: now reaches C90.1, U35.28 (CTX1+)
- net USBM2_TXN: now reaches C93.1, U35.30 (CTX2-)
- net USBM2_TXP: now reaches C91.1, U35.31 (CTX2+)
- net at R45.1: no longer U8.30 (GPIO19)
- net at R46.1: now also U39.4 (IO0)
- net DISP_BACKLIGHT_3V3: now reaches C105.1, J13.28 (Pin_28), J13.29 (Pin_29), J13.30 (Pin_30), J13.31 (Pin_31), J13.5 (Pin_5), J13.6 (Pin_6)
- net DISP_BACKLIGHT_3V3: now also R138.2, U36.1 (OUT)
- net 1V1_ENABLE: no longer names the net of U8.35 (GPIO23)
- net 3V3_ENABLE: no longer names the net of U8.36 (GPIO24)
- net BACKLIGHT_EN renamed DISP_1BL_2EN
- net DISP_EN renamed DISP_2_PWM
- net DISP_2_PWM: now also R139.1
- net DISP_EN_L renamed DISP_1EN_2BL
- net DISP_1EN_2BL: now also R46.2, R138.1, R139.2
- net DISP_TE: no longer names the net of J13.7 (Pin_7)
- new net: R129.1, U36.5 (ISET)
- new net: R137.2, U39.13 (~{RESET})
- new net: C145.1, R133.2, U37.10 (VCC)
- new net: TP7.1, U38.11 (SUSPEND)
- new net: R132.2, U39.1 (A0)
- new net: TP8.1, U38.12 (WAKEUP)
- new net: C147.1, U38.16 (VCCD)
- new net: TP9.1, U38.31 (GPIO_6)
- new net: R128.1, U36.3 (FLG)
- new net DISP_BL_PWR_EN_L: R130.2, U36.4 (EN), U39.10 (IO5)
- new net KICKSTART: R44.2, R45.2, SW3.1 (A)
- new net UART_U+: U37.3 (D2+), U38.14 (USBDP)
- new net UART_U-: U37.7 (D2-), U38.15 (USBDM)
- new net USB_P1_DN: J14.A7 (D-), J14.B7 (D-), U15.4 (IO3), U15.7 (IO3), U37.6 (D-)
- new net USB_P1_DP: J14.A6 (D+), J14.B6 (D+), U15.5 (IO4), U15.6 (IO4), U37.4 (D+)
- new net USB_UART_3V3: C146.1, R134.1, R135.1, R136.1, U38.1 (VDDD), U38.19 (VBUS), U38.23 (VDDD)
- new net USWITCH_4: R118.2, R131.1, U37.1 (S)
- no-connect marks 205 -> 218
Other:
- note added: "External port 1 USB 2.0"
- note added: "GPIO bank controlled via I2C by System Controller"
- note added: "P0 is open drain!"
- note added: "Pol. swap"
- note added: "Sysctl GPIO Bank"
- note added: "TODO: 0.2uF?"
- note added: "TODO: 3v3 power switch here!"
- note added: "TODO: confirm this is good, pulls?"
- note added: "TODO: fix nvme mount position"
- note added: "TODO: move to sysctl"
- note added: "TODO: spi test points"
- note added: "TODO: split these signals?"
- note added: "note: cap only connection"
- note added: "note: confirm pinout/footprint (tssop vs qfn)"
- note added: "on V1: power enables"
- note added: "on display v1: HiZ on display v2: PWM the backlight (overpower R138)"
- note added: "on display v2: HiZ on display v1: low to turn off display"
- note removed: "Latch for Enables"
- note removed: "Power rail switches"
- note removed: "TODO: S_3V3 caps"
- note removed: "TODO: replace with i2c solution from next?"
- note removed: "TODO: serial ports are inconvenient. add USB-uart from classic? SBU+breakout? jst behind port cover?"
- moved on the sheet: C129, C131, C90, C91, C92, C93, R115, R118, R122, R123, R124, R63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

Commit message: mb1.5: small schematic updates
Parts:
- removed J61: UART, Connector_JST:JST_SH_SM04B-SRSS-TB_1x04-1MP_P1.00mm_Horizontal, symbol Connector_Generic:Conn_01x04
- added TP1, TP2, TP3, TP4: TestPoint, TestPoint:TestPoint_Pad_D1.0mm, symbol Connector:TestPoint
- C22, C24, C26, C36: footprint Capacitor_SMD:C_0603_1608Metric -> Capacitor_SMD:C_0402_1005Metric
- C34: value 1uF -> 0.1uF; footprint Capacitor_SMD:C_0603_1608Metric -> Capacitor_SMD:C_0402_1005Metric; LCSC C15849 -> (none); Manufacturer Samsung -> (none); Manufacturer_No CL10A105KB8NNNC -> (none)
- C41: value 1uF -> 4.7uF; footprint Capacitor_SMD:C_0603_1608Metric -> Capacitor_SMD:C_0402_1005Metric; LCSC C15849 -> (none); Manufacturer Samsung -> (none); Manufacturer_No CL10A105KB8NNNC -> (none)
- SW1: footprint Button_Switch_SMD:SW_DIP_SPSTx01_Slide_Omron_A6S-110x_W8.9mm_P2.54mm -> Button_Switch_SMD:SW_DIP_SPSTx01_Slide_Copal_CHS-01A_W5.08mm_P1.27mm_JPin
Connections:
- net GND: now also TP3.1
- net SWC: now also TP2.1
- net SWD: now also TP4.1
- net VCC: now also C30.1, TP1.1
- net SYSLED_G: now reaches R58.1, U8.28 (GPIO17)
- net RRUD-: now reaches R48.1, U8.46 (USB_DM)
- net SYSLED_B: now reaches R61.1, U8.18 (GPIO15)
- net at C26.1, C28.1, C29.1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: no longer C30.1
- net SYSLED_R: now reaches R60.1, U8.27 (GPIO16)
- net R_USB_SRC_EN: now reaches R33.1, U8.40 (GPIO28_ADC2)
- net RRUD+: now reaches R47.1, U8.47 (USB_DP)
- net PWREN_LATCH: no longer names the net of U8.41 (GPIO29_ADC3)
- no-connect marks 218 -> 219
Other:
- moved on the sheet: C25, C26, C27, C28, R47, R48

Commit message: mb1.5 WIP
Connections:
- net VCC: no longer C11.1, C12.1, C129.1, C13.2, C130.1, C131.1, C135.1, C142.1, C143.1, C144.1, C148.1, C2.1, C25.1, C27.1, C30.1, C31.1, C32.1, C33.1, C34.1, C35.1, C36.1, C40.1, C46.2, C5.1, C7.1, C8.1, D5.1 (K), J1.5 (Pin_5), J20.2 (Pin_2), J5.1 (Pin_1), L1.2, R111.2, R113.1, R114.1, R117.2, R119.2, R127.2, R131.2, R132.1, R133.1, R137.1, R19.2, R38.1, R44.1, R56.1, R57.2, R59.2, R72.1, R9.2, TP1.1, U10.8 (VCC), U11.8 (VDD), U2.10 (VCC), U23.3 (VDD), U23.4 (VDD), U29.10 (VOS), U29.2 (VIN), U30.10 (VCC), U31.10 (VCC), U32.6 (IN), U33.4 (VCC), U34.8 (VDD), U39.14 (VDD), U5.6 (OUT), U6.14 (VIN1), U6.2 (VIN2), U8.1 (IOVDD), U8.10 (IOVDD), U8.22 (IOVDD), U8.33 (IOVDD), U8.42 (IOVDD), U8.43 (ADC_AVDD), U8.44 (VREG_IN), U8.48 (USB_VDD), U8.49 (IOVDD)
- new net STANDBY_3V3: C13.2, C130.1, C131.1, C135.1, C142.1, C143.1, C144.1, C148.1, C25.1, C27.1, C30.1, C31.1, C32.1, C33.1, C34.1, C35.1, C36.1, C40.1, C46.2, J1.5 (Pin_5), J20.2 (Pin_2), J5.1 (Pin_1), L1.2, R111.2, R113.1, R114.1, R117.2, R127.2, R131.2, R132.1, R133.1, R137.1, R19.2, R38.1, R44.1, R56.1, R57.2, R59.2, R9.2, TP1.1, U10.8 (VCC), U11.8 (VDD), U2.10 (VCC), U23.3 (VDD), U23.4 (VDD), U29.10 (VOS), U30.10 (VCC), U31.10 (VCC), U33.4 (VCC), U34.8 (VDD), U39.14 (VDD), U8.1 (IOVDD), U8.10 (IOVDD), U8.22 (IOVDD), U8.33 (IOVDD), U8.42 (IOVDD), U8.43 (ADC_AVDD), U8.44 (VREG_IN), U8.48 (USB_VDD), U8.49 (IOVDD)
- new net SYS_VCC: C11.1, C12.1, C129.1, C2.1, C5.1, C7.1, C8.1, D5.1 (K), R119.2, R72.1, U29.2 (VIN), U32.6 (IN), U5.6 (OUT), U6.14 (VIN1), U6.2 (VIN2)
Other:
- note added: "TODO FIX"
- note added: "TODO: unconnected"
- note removed: "TODO: serial to SBU?"
- moved on the sheet: C13, C56, C62, D3, FB2, H8, H9, R10, R100, R14, R69, R97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
